Commit message: Align UR5e mount nozzle and print path

File: robotic_printing_platform/robots/robot_configs/ur5e/robot.urdf (robot description, URDF)
Before this commit: robot universal_robots_ur5e_planning, 14 links, 13 joints
Links:
- removed link elbow_rot
- removed link shoulder_lift_rot
- removed link shoulder_pan_rot
- removed link wrist_1_rot
- removed link wrist_2_rot
- removed link wrist_3_rot
- added link base_link_inertia
- added link flange
Joints:
- removed joint elbow_fixed
- removed joint flange_to_tool0
- removed joint shoulder_lift_fixed
- removed joint shoulder_pan_fixed
- removed joint wrist_1_fixed
- removed joint wrist_2_fixed
- removed joint wrist_3_fixed
- added joint base_link-base_link_inertia: type fixed, parent base_link, child base_link_inertia, origin xyz=0 0 0 rpy=0 0 3.141592653589793
- added joint flange-tool0: type fixed, parent flange, child tool0, origin xyz=0 0 0 rpy=1.5707963267948966 0 1.5707963267948966
- added joint wrist_3-flange: type fixed, parent wrist_3_link, child flange, origin xyz=0 0 0 rpy=0 -1.5707963267948966 -1.5707963267948966
- joint elbow_joint: child elbow_rot -> forearm_link; origin xyz=0 0 0 rpy=0 0 0 -> xyz=-0.425 0 0 rpy=0 0 0
- joint shoulder_lift_joint: child shoulder_lift_rot -> upper_arm_link; origin xyz=0 0 0 rpy=0 0 0 -> xyz=0 0 0 rpy=1.5707963267948966 0 0
- joint shoulder_pan_joint: child shoulder_pan_rot -> shoulder_link; parent base_link -> base_link_inertia
- joint wrist_1_joint: child wrist_1_rot -> wrist_1_link; origin xyz=0 0 0.1333 rpy=0 0 0 -> xyz=-0.3922 0 0.1333 rpy=0 0 0
- joint wrist_2_joint: child wrist_2_rot -> wrist_2_link; origin xyz=0 0 0.0997 rpy=0 0 0 -> xyz=0 -0.0997 0 rpy=1.5707963267948966 0 0
- joint wrist_3_joint: child wrist_3_rot -> wrist_3_link; origin xyz=0 0 0.0996 rpy=0 0 0 -> xyz=0 0.0996 0 rpy=1.5707963267948966 3.141592653589793 3.141592653589793
